File: design/v1/CPU.kicad_sch (KiCad schematic)
At the start: 11 parts, among them IC1 MC68030RC_PGA, Q2 5H8ET-20.000

Commit message: Tidy up readme
Connections:
- net HALT is gone; now on net RESET: IC1.H2 (HLT)
Changed lines of the file:
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@@
+	)
+	(junction
+		(at 40.64 55.88)
+		(diameter 0)
+		(color 0 0 0 0)
 	)
 	(junction
@@
 	(wire
 		(pts
+			(xy 40.64 53.34) (xy 40.64 55.88)
+		)
+		(stroke
+			(width 0)
+			(type default)
+		)
+	)
+	(wire
+		(pts
 			(xy 62.23 24.13) (xy 64.77 24.13)
 		)
@@
 		(pts
 			(xy 62.23 33.02) (xy 62.23 24.13)
+		)
+		(stroke
+			(width 0)
+			(type default)
+		)
+	)
+	(wire
+		(pts
+			(xy 39.37 55.88) (xy 40.64 55.88)
 		)
 		(stroke
@@
 	(global_label "RESET"
 		(shape bidirectional)
-		(at 40.64 55.88 180)
-		(fields_autoplaced yes)
-		(effects
-			(font
-				(size 1.27 1.27)
-			)
-			(justify right)
-		)
-		(property "Intersheetrefs" "${INTERSHEET_REFS}"
-			(at -5.08 1.27 0)
+		(at 39.37 55.88 180)
+		(fields_autoplaced yes)
+		(effects
+			(font
+				(size 1.27 1.27)
+			)
+			(justify right)
+		)
+		(property "Intersheetrefs" "${INTERSHEET_REFS}"
+			(at -6.35 1.27 0)
 			(effects
 				(font
@@
 		(fields_autoplaced yes)
 		(effects
-			(font
-				(size 1.27 1.27)
-			)
-			(justify right)
-		)
-		(property "Intersheetrefs" "${INTERSHEET_REFS}"
-			(at -5.08 1.27 0)
-			(effects
-				(font
-					(size 1.27 1.27)
-				)
-				(hide yes)
-			)
-		)
-	)
-	(global_label "HALT"
-		(shape input)
-		(at 40.64 53.34 180)
-		(fields_autoplaced yes)
-		(effects
